Commit message: urdf base_footprint imu_link changed

File: src/robot_description/urdf/platform_base_allink.urdf (robot description, URDF)
Before this commit: robot platform_base_allink, 7 links, 6 joints
Links:
- removed link IMU_link
- added link imu_link, mass 0.001; collision mesh filename=package://robot_description/meshes/IMU_link.STL; visual mesh filename=package://robot_description/meshes/IMU_link.STL
Joints:
- joint IMU_joint: child IMU_link -> imu_link; origin xyz=-0.195 0 0.695 rpy=0 0 0 -> xyz=-0.195 0 0.695 rpy=0 0 -1.5708
- joint base_foot_joint: child base_footprint -> base_link; origin xyz=0 0 -0.274 rpy=0 0 0 -> xyz=0 0 0.274 rpy=0 0 0; parent base_link -> base_footprint

Commit message: seong jae

File: src/robot_description/urdf/platform_base_allink.urdf (robot description, URDF)
Before this commit: robot platform_base_allink, 6 links, 5 joints
Links:
- added link base_foot_link, mass 0.001
Joints:
- added joint odom: type continuous, parent base_link, child base_foot_link, origin xyz=0 0 -0.274 rpy=0 0 0, axis 0 0 1
- joint GPS_joint: origin xyz=0 -0.195 0.545 rpy=0 0 1.5708 -> xyz=0 -0.195 0.835 rpy=0 0 0
- joint IMU_joint: origin xyz=0 -0.195 0.545 rpy=0 0 1.5708 -> xyz=0 -0.195 0.695 rpy=0 0 0
- joint base_foot_joint: origin xyz=0 0 -0.274 rpy=0 0 1.5708 -> xyz=0 0 -0.274 rpy=0 0 0
- joint camera_joint: origin xyz=0 0.42 0.545 rpy=0 0 1.5708 -> xyz=0 0.42 0.545 rpy=0 0 0
- joint laser_joint: origin xyz=0 0 0.695 rpy=0 0 1.5708 -> xyz=0 0 0.695 rpy=0 0 0

Commit message: modified urdf file

File: src/robot_description/urdf/platform_base_allink.urdf (robot description, URDF)
Before this commit: robot platform_base_allink, 7 links, 6 joints
Joints:
- joint GPS_joint: origin xyz=0 -0.195 0.835 rpy=0 0 0 -> xyz=-0.195 0 0.835 rpy=0 0 0
- joint IMU_joint: origin xyz=0 -0.195 0.695 rpy=0 0 0 -> xyz=-0.195 0 0.695 rpy=0 0 0
- joint camera_joint: origin xyz=0 0.42 0.545 rpy=0 0 0 -> xyz=0.42 0 0.545 rpy=0 0 0

Commit message: amcl add

File: src/robot_description/urdf/platform_base_allink.urdf (robot description, URDF)
Before this commit: robot platform_base_allink, 7 links, 6 joints
Links:
- removed link laser_link
- added link velodyne, mass 0.001; collision mesh filename=package://robot_description/meshes/laser_link.STL; visual mesh filename=package://robot_description/meshes/laser_link.STL
Joints:
- joint laser_joint: child laser_link -> velodyne
