Commit message: transfer

File: robot_description/urdf/platform_base_allink.urdf (robot description, URDF)
Before this commit: robot platform_base_allink, 7 links, 6 joints
Joints:
- joint IMU_joint: origin xyz=-0.195 0 0.695 rpy=0 0 -1.5708 -> xyz=-0.195 0 0.695 rpy=0 3.14 0

Commit message: navigation_state_machine

File: robot_description/urdf/platform_base_allink.urdf (robot description, URDF)
Before this commit: robot platform_base_allink, 7 links, 6 joints
Links:
- removed link base_foot_link
- link base_footprint: mass 0.001 -> None; geometry 
Joints:
- removed joint base_foot_joint
- removed joint odom
- added joint base_joint: type fixed, parent base_footprint, child base_link, origin xyz=0.0 0.0 0.40 rpy=0 0 0
